File: Kicad/phaseB.kicad_sch (KiCad schematic)
At the start: 47 parts, among them J1 USB_B_Mini, J2 AVR-ISP-6, U1 CA56-12EWA, U2 74HC595, U3 ATmega32U4-A, U4 USBLC6-2SC6, U5 LP2985-3.3, Y1 Crystal_GND24

Commit message: emb
layout and stuff
Parts:
- removed C1, C2: 22pF, Capacitor_SMD:C_0603_1608Metric, symbol Device:C
- removed C10, C14: 1uF, Capacitor_SMD:C_0603_1608Metric, symbol Device:C
- removed C11, C4, C5, C6, C7, C8, C9: 0.1uF, Capacitor_SMD:C_0603_1608Metric, symbol Device:C
- removed C12: 10nF, Capacitor_SMD:C_0603_1608Metric, symbol Device:C
- removed C13: 2.2uF, Capacitor_SMD:C_0603_1608Metric, symbol Device:C
- removed C3: 10uF, Capacitor_SMD:C_0603_1608Metric, symbol Device:C
- removed J1: USB_B_Mini, Connector_USB:USB_Mini-B_Lumberg_2486_01_Horizontal, symbol Connector:USB_B_Mini
- removed J2: AVR-ISP-6, Connector_PinSocket_2.54mm:PinSocket_2x03_P2.54mm_Vertical, symbol Connector:AVR-ISP-6
- added C1: 0.1u, Capacitor_SMD:C_0603_1608Metric, symbol Device:C_Small
- added C10, C11, C12, C4, C5, C6, C7: 0.1uF, Capacitor_SMD:C_0603_1608Metric, symbol Device:C_Small
- added C13, C9: 1uF, Capacitor_SMD:C_0603_1608Metric, symbol Device:C_Small
- added C14: 2.2uF, Capacitor_SMD:C_0603_1608Metric, symbol Device:C_Small
- added C2, C3: 22p, Capacitor_SMD:C_0603_1608Metric, symbol Device:C_Small
- added C8: 10uF, Capacitor_SMD:C_0805_2012Metric, symbol Device:C_Polarized_Small_US
- added J1: AVR-ISP-6, Connector_PinSocket_2.54mm:PinSocket_2x03_P2.54mm_Vertical, symbol Connector:AVR-ISP-6
- added J2: USB_B_Mini, Connector_USB:USB_Mini-B_Lumberg_2486_01_Horizontal, symbol Connector:USB_B_Mini
- added J3: ESP_Conn, Connector_PinSocket_2.54mm:PinSocket_2x04_P2.54mm_Vertical, symbol Connector_Generic:Conn_02x04_Odd_Even
- added R17: 10k, Resistor_SMD:R_0603_1608Metric, symbol Device:R_Small
- C15: value 0.1u -> 10nF
- F1: value PTVSD? -> PTCSMD
- R1, R2: footprint Resistor_SMD:R_0603_1608Metric -> Resistor_SMD:R_0805_2012Metric
- R14: value 1k -> 22; footprint Resistor_SMD:R_0805_2012Metric -> Resistor_SMD:R_0603_1608Metric
- R16: value 22 -> 1k
- Y1: value Crystal_GND24 -> 16MHz
Connections:
- net +3.3V: now also C14.1, J3.4 (Pin_4), J3.6 (Pin_6), J3.8 (Pin_8), R17.1
- net +5V: now also R16.1, C1.1, C10.1, C11.1, C13.1, C4.1, C5.1, C6.1, C7.1, C8.1, J1.2 (VCC); no longer C15.1, R14.1
- net AREF: now also C12.1
- net GND: now also C1.2, C10.2, C11.2, C12.2, C13.2, C14.2, C2.1, C3.2, C4.2, C5.2, C6.2, C7.2, C8.2, C9.2, J1.6 (GND), J2.5 (GND), J3.1 (Pin_1)
- net MISO: now also J1.1 (MISO)
- net MOSI: now also J1.4 (MOSI)
- net RST: now also J1.5 (~{RST})
- net RX: now also J3.7 (Pin_7)
- net SCK: now also J1.3 (SCK)
- net TX: now also J3.2 (Pin_2)
- net UCAP: now also C9.1
- net USB_CONN_D+: now also R14.2; no longer R15.2
- net USB_CONN_D-: now also R15.2; no longer R16.2
- net XTAL1: now also C2.2
- net XTAL2: now also C3.1
- net at D3.2 (A): now also R16.2; no longer R14.2
- net at R15.1: now also J2.2 (D-)
- net at F1.1: now also J2.1 (VBUS)
- net at U5.4 (BP): now also C15.1
- new net: J2.3 (D+), R14.1
- new net: J3.5 (Pin_5), R17.2
- no-connect marks 15 -> 16
Other:
- note added: "ATMEGA32U4"
- note added: "ESP8266 Conn"
- note removed: "Cade Thornton"
- note removed: "Crystal"
- note removed: "Microprocessor"
- note removed: "Power indicator"
- note removed: "Reset Button"
- note removed: "USB Connector"
- title: Arduino Uno Shield -> ATMEGA Kitchen Timer
- moved on the sheet: D1, D2, LS1, R1, R10, R11, R12, R2, R3, R4, R5, R6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
