File: Kicad/phaseB.kicad_pcb (KiCad board)
At the start: 2 copper layers, 95 x 77 mm, 53 parts, among them J1 AVR-ISP-6, J2 USB_B_Mini, J3 ESP_Conn, M3 MountingHole_3.2mm_M3, U1 CA56-12EWA, U2 74HC595, U3 ATmega32U4-A, U4 USBLC6-2SC6, U5 LP2985-3.3, Y1 16MHz

Commit message: e
e
Other:
- board text added: "CADE T."
- board text added: "Kitchen Timer"
- board text added: "November 2023"
- board text removed: "April 2023"
- board text removed: "Kitchen Timer Version 2"
Changed lines of the file:
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@@
   (gr_line (start 94.920802 140.495) (end 94.920802 63.495)
     (stroke (width 0.2) (type solid)) (layer "Edge.Cuts"))
-  (gr_text "Kitchen Timer Version 2\n\n" (at 154.94 134.62) (layer "F.SilkS")
+  (gr_text "CADE T." (at 167.64 129.54) (layer "F.Cu")
+    (effects (font (size 1.5 1.5) (thickness 0.3) bold) (justify left bottom))
+  )
+  (gr_text "Kitchen Timer\n\n" (at 154.94 134.62) (layer "F.SilkS")
     (effects (font (size 1 1) (thickness 0.15)) (justify left bottom))
   )
@@
     (effects (font (size 1 1) (thickness 0.15)) (justify left bottom))
   )
-  (gr_text "April 2023\n" (at 154.94 134.62) (layer "F.SilkS")
+  (gr_text "November 2023\n" (at 154.94 134.62) (layer "F.SilkS")
     (effects (font (size 1 1) (thickness 0.15)) (justify left bottom))
   )
